Commit message: Migrating to latest  lerobot and adding dual overhead cameras

File: so101_description/urdf/so101_arm.urdf.xacro (robot description, xacro)
@@ -8,16 +8,7 @@
   <xacro:arg name="usb_port" default="/dev/ttyUSB0"/>
   <xacro:arg name="joint_config_file" default=""/>
-  <!-- Camera args -->
-  <xacro:arg name="enable_static_cam" default="false"/>
-  <xacro:arg name="enable_wrist_cam" default="false"/>
-  <xacro:arg name="cam_static_xyz" default="0.2 0.0 0.60"/>
-  <xacro:arg name="cam_static_rpy" default="0.0 1.5708 0.0"/>
-  <xacro:arg name="cam_wrist_xyz" default="0.0 0.0 -0.02"/>
-  <xacro:arg name="cam_wrist_rpy" default="-1.5708 0.0 -1.5708"/>
   <!-- Convert args to properties for use in ${} expressions -->
   <xacro:property name="use_ros2_control" value="$(arg use_ros2_control)"/>
   <xacro:property name="variant" value="$(arg variant)"/>
-  <xacro:property name="enable_static_cam" value="$(arg enable_static_cam)"/>
-  <xacro:property name="enable_wrist_cam" value="$(arg enable_wrist_cam)"/>
   <xacro:include filename="$(find so101_description)/urdf/so101_macros.xacro"/>
   <xacro:include filename="$(find so101_description)/urdf/so101_materials.xacro"/>
@@ -50,14 +41,5 @@
       system_name="SO101_${variant}_SYSTEM"/>
   </xacro:if>
-  <!-- Cameras (opt-in via enable_static_cam / enable_wrist_cam) -->
-  <xacro:if value="${enable_static_cam}">
-    <xacro:so101_static_camera
-      xyz="$(arg cam_static_xyz)"
-      rpy="$(arg cam_static_rpy)"/>
-  </xacro:if>
-  <xacro:if value="${enable_wrist_cam}">
-    <xacro:so101_wrist_camera
-      xyz="$(arg cam_wrist_xyz)"
-      rpy="$(arg cam_wrist_rpy)"/>
-  </xacro:if>
+  <!-- The wrist mount is part of the robot. Overhead extrinsics come from the external camera rig. -->
+  <xacro:so101_wrist_camera/>
 </robot>

File: so101_description/urdf/so101_cameras.xacro (robot description, xacro)
@@ -3,39 +3,9 @@
   <!--
     Camera frames for SO-101 arm.
-    Defines static (overhead) and wrist camera links/joints.
-    Position and orientation are configurable via macro params,
-    passed from launch args so each user can match their physical
-    camera mounting.
-    Usage at launch time:
-      xacro ... enable_static_cam:=true cam_static_xyz:="0.2 0.0 0.60"
+    Defines the wrist camera links/joints. Static overhead cameras are
+    external to the robot model and are published from the validated rig file.
     For simulation (Gazebo/MuJoCo), pass include_inertia:=true to avoid
     warnings about links with no inertia.
   -->
-  <xacro:macro name="so101_static_camera"
-               params="xyz:='0.2 0.0 0.60'
-                       rpy:='0.0 1.5708 0.0'
-                       parent:='base_link'
-                       include_inertia:='false'">
-    <link name="static_camera_link">
-      <xacro:if value="${include_inertia}">
-        <inertial>
-          <mass value="0.001"/>
-          <inertia ixx="1e-7" ixy="0" ixz="0" iyy="1e-7" iyz="0" izz="1e-7"/>
-        </inertial>
-      </xacro:if>
-    </link>
-    <joint name="static_camera_joint" type="fixed">
-      <origin xyz="${xyz}" rpy="${rpy}"/>
-      <parent link="${parent}"/>
-      <child link="static_camera_link"/>
-    </joint>
-    <!-- Optical frame: rotated so Z=forward, X=right, Y=down (OpenCV/REP-103) -->
-    <link name="static_camera_optical_frame"/>
-    <joint name="static_camera_optical_joint" type="fixed">
-      <origin xyz="0 0 0" rpy="${-pi/2} 0 ${-pi/2}"/>
-      <parent link="static_camera_link"/>
-      <child link="static_camera_optical_frame"/>
-    </joint>
-  </xacro:macro>
   <xacro:macro name="so101_wrist_camera"
                params="xyz:='0.0 0.0 -0.02'
