Commit message: Fixeid overhead camera stls

File: so101_description/urdf/end_effectors/so101_ee_follower.xacro (robot description, xacro)
@@ -11,6 +11,20 @@
       <xacro:mesh_vc filename="${mesh_dir}/sts3215_03a_v1.stl"
         xyz="0.0077 0.0001 -0.0234" rpy="-1.5708 -5.19179e-17 -1.66533e-16" material="sts3215"/>
-      <xacro:mesh_vc filename="${mesh_dir}/wrist_roll_follower_so101_v1.stl"
-        xyz="8.32667e-17 -0.000218214 0.000949706" rpy="-3.14159 -5.55112e-17 0" material="3d_printed"/>
+      <!-- Integrated 32x32 UVC wrist-camera mount; source STL units are millimetres. -->
+      <visual>
+        <origin xyz="8.32667e-17 -0.000218214 0.000949706" rpy="-3.14159 -5.55112e-17 0"/>
+        <geometry>
+          <mesh filename="${mesh_dir}/wrist_cam_mount_32x32_uvc_so101.stl"
+            scale="0.001 0.001 0.001"/>
+        </geometry>
+        <material name="3d_printed"/>
+      </visual>
+      <!-- Keep the original wrist-roll collision mesh to avoid a dense camera-mount collider. -->
+      <collision>
+        <origin xyz="8.32667e-17 -0.000218214 0.000949706" rpy="-3.14159 -5.55112e-17 0"/>
+        <geometry>
+          <mesh filename="${mesh_dir}/wrist_roll_follower_so101_v1.stl"/>
+        </geometry>
+      </collision>
     </link>
     <xacro:so101_gripper_frame />

File: so101_description/urdf/so101_cameras.xacro (robot description, xacro)
@@ -9,6 +9,6 @@
   -->
   <xacro:macro name="so101_wrist_camera"
-               params="xyz:='0.0202 0.0388 -0.0234'
-                       rpy:='0.0 1.5708 0.0'
+               params="xyz:='0.0025 -0.0720574 0.0041503'
+                       rpy:='1.5707963 1.1344640 1.5707963'
                        parent:='gripper_link'
                        include_inertia:='false'">

Commit message: Improing graspreward function

File: so101_description/urdf/end_effectors/so101_ee_follower.xacro (robot description, xacro)
@@ -2,5 +2,5 @@
 <robot xmlns:xacro="http://www.ros.org/wiki/xacro">
   <xacro:macro name="so101_ee_follower"
-               params="mesh_dir:='package://so101_description/meshes' add_transmissions:='false'">
+               params="mesh_dir:='package://so101_description/meshes' add_transmissions:='false' simulation_contact_pads:='false'">
     <link name="gripper_link">
       <xacro:inertial_block
@@ -45,4 +45,48 @@
       <limit effort="10" velocity="10" lower="-0.174533" upper="1.74533"/>
     </joint>
+    <!--
+      Simulation-only, collision-only contact pads.  Each pad is a distinct fixed
+      rigid body so PhysX contact sensors can distinguish the two jaw faces.
+      The 0.5 mm pad is centred 0.25 mm behind its contact face; the face itself
+      protrudes 0.1 mm beyond the corresponding jaw mesh.
+    -->
+    <xacro:if value="${simulation_contact_pads}">
+      <link name="fixed_jaw_contact_pad_link">
+        <xacro:inertial_block
+          xyz="0 0 0" rpy="0 0 0"
+          mass="0.0001"
+          ixx="7.908333333e-09" ixy="0" ixz="0"
+          iyy="5.210416667e-09" iyz="0" izz="2.702083333e-09"/>
+        <collision>
+          <origin xyz="0 0 0" rpy="0 0 0"/>
+          <geometry>
+            <box size="0.0005 0.018 0.025"/>
+          </geometry>
+        </collision>
+      </link>
+      <joint name="fixed_jaw_contact_pad_joint" type="fixed">
+        <origin xyz="-0.00805 -0.000218 -0.0925" rpy="0 0 0"/>
+        <parent link="gripper_link"/>
+        <child link="fixed_jaw_contact_pad_link"/>
+      </joint>
+      <link name="moving_jaw_contact_pad_link">
+        <xacro:inertial_block
+          xyz="0 0 0" rpy="0 0 0"
+          mass="0.0001"
+          ixx="7.908333333e-09" ixy="0" ixz="0"
+          iyy="2.702083333e-09" iyz="0" izz="5.210416667e-09"/>
+        <collision>
+          <origin xyz="0 0 0" rpy="0 0 0"/>
+          <geometry>
+            <box size="0.0005 0.025 0.018"/>
+          </geometry>
+        </collision>
+      </link>
+      <joint name="moving_jaw_contact_pad_joint" type="fixed">
+        <origin xyz="-0.01215 -0.0691 0.0190" rpy="0 0 0"/>
+        <parent link="moving_jaw_so101_v1_link"/>
+        <child link="moving_jaw_contact_pad_link"/>
+      </joint>
+    </xacro:if>
     <!-- follower-only motor6 transmission (optional) -->
     <xacro:if value="${add_transmissions}">

File: so101_description/urdf/so101_arm.urdf.xacro (robot description, xacro)
@@ -4,4 +4,5 @@
   <xacro:arg name="mesh_dir" default="package://so101_description/meshes"/>
   <xacro:arg name="add_transmissions" default="false"/>
+  <xacro:arg name="simulation_contact_pads" default="false"/>
   <xacro:arg name="use_ros2_control" default="false"/>
   <xacro:arg name="hardware_type" default="mock"/>
@@ -30,5 +31,6 @@
     <xacro:so101_ee_follower
       mesh_dir="$(arg mesh_dir)"
-      add_transmissions="$(arg add_transmissions)"/>
+      add_transmissions="$(arg add_transmissions)"
+      simulation_contact_pads="$(arg simulation_contact_pads)"/>
   </xacro:if>
   <xacro:if value="${use_ros2_control}">

Commit message: Fixing reward for gripper

File: so101_description/urdf/end_effectors/so101_ee_follower.xacro (robot description, xacro)
@@ -20,5 +20,13 @@
         <material name="3d_printed"/>
       </visual>
-      <!-- Keep the original wrist-roll collision mesh to avoid a dense camera-mount collider. -->
+      <!-- Fixed-jaw finger: visible AND collision so the cameras render the real
+           gripping surface (at the contact pad) instead of only the camera bracket. -->
+      <visual>
+        <origin xyz="8.32667e-17 -0.000218214 0.000949706" rpy="-3.14159 -5.55112e-17 0"/>
+        <geometry>
+          <mesh filename="${mesh_dir}/wrist_roll_follower_so101_v1.stl"/>
+        </geometry>
+        <material name="3d_printed"/>
+      </visual>
       <collision>
         <origin xyz="8.32667e-17 -0.000218214 0.000949706" rpy="-3.14159 -5.55112e-17 0"/>
@@ -84,5 +92,8 @@
       </link>
       <joint name="moving_jaw_contact_pad_joint" type="fixed">
-        <origin xyz="-0.01215 -0.0691 0.0190" rpy="0 0 0"/>
+        <!-- Origin X calibrated so the pad face is flush with the moving-jaw
+             finger mesh at the grasp angle (pad protrudes ~0.1 mm, not the
+             ~2.7 mm invisible gap produced by the previous -0.01215 value). -->
+        <origin xyz="-0.00996 -0.0691 0.0190" rpy="0 0 0"/>
         <parent link="moving_jaw_so101_v1_link"/>
         <child link="moving_jaw_contact_pad_link"/>
